Commit message: 夹取老虎（viser左部有一点页面

File: data/ur5e_robotiq/ur5e_isaaclab.urdf (robot description, URDF)
Before this commit: robot ur5e, 10 links, 9 joints
Links:
- link base_link: geometry visual mesh filename=../ur7e_description/meshes/obj/base_link.obj
- link forearm_link: geometry visual mesh filename=../ur7e_description/meshes/obj/forearm_link.obj
- link shoulder_link: geometry visual mesh filename=../ur7e_description/meshes/obj/shoulder_link.obj
- link upper_arm_link: geometry visual mesh filename=../ur7e_description/meshes/obj/upper_arm_link.obj
- link wrist_1_link: geometry visual mesh filename=../ur7e_description/meshes/obj/wrist_1_link.obj
- link wrist_2_link: geometry visual mesh filename=../ur7e_description/meshes/obj/wrist_2_link.obj
- link wrist_3_link: geometry visual mesh filename=../ur7e_description/meshes/obj/wrist_3_link.obj
